File: PCB/Mainboard/V1/mainboard_v1/mainboard_v1.sch (KiCad schematic (older format))
At the start: 46 parts, among them J1 22-23-2021, J2 USB_B_Micro, J3 527450697, J4 527450697, J5 M50-3100545, J6 M50-3100545, J7 M50-3100545, SW1 SW_SPDT, U1 MDBT50Q-1MV2, U3 MCP73831T-2ACI_OT, U4 AP2112K-3.3, U5 MPU6050

Commit message: udated by FZ
Parts:
- removed C13, C9: 10uF, Capacitor_SMD:C_0603_1608Metric_Pad1.08x0.95mm_HandSolder, symbol Device:C_Small
- removed H4: M2, Mylib:mounthole_1.8mm, symbol Mechanical:MountingHole
- removed H5, H6: M2, Mylib:M2_NPTH_mounting_hole, symbol Mechanical:MountingHole
- removed J3, J4: 527450697, symbol Mylib:527450697
- removed J6: M50-3100545, SnapEDA Library:HARWIN_M50-3100545, symbol M50-3100545:M50-3100545
- added C13, C9: TAJP106K010RNJ, SamacSys_Parts:CAPPM2014X170N, symbol SamacSys_Parts:TAJP106K010RNJ
- added C14, C15, C16, C17: 10uF, Capacitor_SMD:C_0603_1608Metric_Pad1.08x0.95mm_HandSolder, symbol Device:C_Small
- added C18: 0.1uF, Capacitor_SMD:C_0603_1608Metric_Pad1.08x0.95mm_HandSolder, symbol Device:C_Small
- added IC1, IC2: MP6513GJ-Z, SamacSys_Parts:SOT95P280X100-6N, symbol SamacSys_Parts:MP6513GJ-Z
- added J10, J11, J12, J13, J14, J15, J16, J17, J18, J19, J20, J9: 1_pin_sig, Mylib:1.27mm_pin_hole, symbol Mylib:1_pin_sig
- added J3, J8: 1734592-6, SamacSys_Parts:17345926, symbol SamacSys_Parts:1734592-6
- added J4: 22-23-2021, Connector_PinHeader_1.27mm:PinHeader_2x01_P1.27mm_Vertical, symbol dk_Rectangular-Connectors-Headers-Male-Pins:22-23-2021
- added J6: 20021321-00014C1LF, SamacSys_Parts:2002132100014C1LF, symbol SamacSys_Parts:20021321-00014C1LF
- added R10, R11: 10k, Resistor_SMD:R_0603_1608Metric_Pad0.98x0.95mm_HandSolder, symbol Device:R_Small
- added S1: B3U-1000P, digikey-footprints:Switch_Tactile_SMD_B3U-1000P, symbol dk_Tactile-Switches:B3U-1000P
- added U7: AP2112K-3.3, Package_TO_SOT_SMD:SOT-23-5_HandSoldering, symbol Regulator_Linear:AP2112K-3.3
- C12, C8: value 10uF -> 0.1uF
- C2: value 0.1uF -> 10uF
- J5, J7: value M50-3100545 -> 20021321-00010C4LF
- R6: value 10k -> 4.99k
- XTAL1: footprint digikey-footprints:SMD-2_3.2x1.5mm -> SamacSys_Parts:ECS32712512TR
Connections:
- net labels added: A0, A1, A3, A4, A5, D10, D11, D12, D13, D2, D5, D6, D9, M1_IN1, M1_IN2, M1_O1, M1_O2, M2_IN1, M2_IN2, M2_O1, M2_O2, RXD, SWO, TXD, VCC
- net labels removed: ADC_BAT, FAULT_1, FAULT_2, MOTOR_1_IN1, MOTOR_1_IN2, MOTOR_1_O1, MOTOR_1_O2, MOTOR_2_IN1, MOTOR_2_IN2, MOTOR_2_O1, MOTOR_2_O2
- wire segments 185 -> 266
- no-connect marks 18 -> 35
Other:
- moved on the sheet: C10, C11, C12, C2, C5, C6, C8, D1, D2, D3, D4, H1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

Commit message: udated by FZ
Connections:
- net labels added: GP0, GP1, GP2, GP3, MOTOR1_A, MOTOR1_B
- net labels removed: A4, D2
- wire segments 266 -> 268
- no-connect marks 35 -> 36
Other:
- moved on the sheet: D3, J20, R5
Changed lines of the file:
@@
 	2050 4300 1700 4300
-Wire Wire Line
-	4250 3800 4550 3800
 Wire Wire Line
 	4250 3700 4550 3700
@@
 L Device:LED D3
 U 1 1 61242DE4
-P 5550 5550
-F 0 "D3" V 5497 5630 50  0000 L CNN
-F 1 "LED" V 5588 5630 50  0000 L CNN
-F 2 "LED_SMD:LED_0603_1608Metric_Pad1.05x0.95mm_HandSolder" H 5550 5550 50  0001 C CNN
-F 3 "~" H 5550 5550 50  0001 C CNN
-	1    5550 5550
+P 5550 5300
+F 0 "D3" V 5497 5380 50  0000 L CNN
+F 1 "LED" V 5588 5380 50  0000 L CNN
+F 2 "LED_SMD:LED_0603_1608Metric_Pad1.05x0.95mm_HandSolder" H 5550 5300 50  0001 C CNN
+F 3 "~" H 5550 5300 50  0001 C CNN
+	1    5550 5300
 	0    1    1    0
 $EndComp
@@
 L Device:R_Small R5
 U 1 1 6124B72D
-P 5550 5250
-F 0 "R5" V 5450 5250 50  0000 C CNN
-F 1 "1k" V 5650 5250 50  0000 C CNN
-F 2 "Resistor_SMD:R_0603_1608Metric_Pad0.98x0.95mm_HandSolder" H 5550 5250 50  0001 C CNN
-F 3 "~" H 5550 5250 50  0001 C CNN
-	1    5550 5250
+P 5550 5600
+F 0 "R5" V 5450 5600 50  0000 C CNN
+F 1 "1k" V 5650 5600 50  0000 C CNN
+F 2 "Resistor_SMD:R_0603_1608Metric_Pad0.98x0.95mm_HandSolder" H 5550 5600 50  0001 C CNN
+F 3 "~" H 5550 5600 50  0001 C CNN
+	1    5550 5600
 	-1   0    0    1
 $EndComp
 Wire Wire Line
-	5550 5400 5550 5350
+	5550 5500 5550 5450
 $Comp
 L power:GND #PWR0122
@@
 NoConn ~ 10100 2050
 NoConn ~ 10100 2250
-NoConn ~ 10100 2450
+NoConn ~ 10100 2650
 NoConn ~ 8300 2250
 NoConn ~ 8300 2350
@@
 	5650 1600 5900 1600
 Wire Wire Line
-	6900 1200 7150 1200
+	6900 1200 6950 1200
 Wire Wire Line
 	7150 1300 6900 1300
@@
 	7150 2550 6900 2550
 Wire Wire Line
-	5850 2150 5900 2150
-Wire Wire Line
 	5650 2250 5900 2250
 Wire Wire Line
@@
 	5650 2450 5900 2450
 Wire Wire Line
-	5650 2550 5900 2550
+	5850 2550 5900 2550
 $Comp
 L power:GND #PWR0139
@@
 	9400 5150 9450 5150
 Wire Wire Line
-	10350 5150 10650 5150
-Wire Wire Line
-	10650 5250 10350 5250
-Wire Wire Line
-	10650 5350 10350 5350
-Wire Wire Line
-	10650 5450 10350 5450
-Wire Wire Line
-	10650 5550 10350 5550
-Wire Wire Line
-	10650 5650 10350 5650
-Wire Wire Line
-	10650 4450 10350 4450
-Wire Wire Line
-	10650 4350 10350 4350
-Wire Wire Line
-	10650 4250 10350 4250
-Wire Wire Line
-	10650 4150 10350 4150
-Wire Wire Line
-	10650 4050 10350 4050
-Wire Wire Line
-	10650 3950 10350 3950
+	10750 5350 10350 5350
+Wire Wire Line
+	10750 5450 10350 5450
+Wire Wire Line
+	10750 4250 10350 4250
+Wire Wire Line
+	10750 4150 10350 4150
 Wire Wire Line
 	5250 3600 5200 3600
@@
 Text Label 8600 5400 2    50   ~ 0
 M2_O2
+Text Label 5650 1600 0    50   ~ 0
+SCL
+Text Label 5650 1400 0    50   ~ 0
+SCK
+Text Label 5650 1500 0    50   ~ 0
+SDA
+Text Label 5650 1300 0    50   ~ 0
+MOSI
 Text Label 5650 1200 0    50   ~ 0
-SCL
-Text Label 5650 1300 0    50   ~ 0
-SCK
-Text Label 5650 1400 0    50   ~ 0
-SDA
-Text Label 5650 1500 0    50   ~ 0
-MOSI
-Text Label 5650 1600 0    50   ~ 0
 MISO
 Text Label 1700 4000 0    50   ~ 0
 A3
-Text Label 7150 1200 2    50   ~ 0
+Text Label 7150 1500 2    50   ~ 0
 A1
 NoConn ~ 4550 3000
@@
 NoConn ~ 4550 2900
 NoConn ~ 4550 2700
-NoConn ~ 4550 4000
 NoConn ~ 4550 2800
 $Comp
@@
 Text Label 1700 1500 0    50   ~ 0
 A5
-Text Label 1700 1400 0    50   ~ 0
-A4
 $Comp
 L Regulator_Linear:AP2112K-3.3 U7
@@
 	0    1    1    0
 $EndComp
+Text Label 4550 3900 2    50   ~ 0
+M1_IN1
 Text Label 4550 4100 2    50   ~ 0
-M1_IN1
-Text Label 1700 4100 0    50   ~ 0
 M1_IN2
 $Comp
@@
 Wire Wire Line
 	7550 4750 7650 4750
-NoConn ~ 1700 4300
-Text Label 5650 2550 0    50   ~ 0
+Text Label 5650 2450 0    50   ~ 0
 A1
 Text Label 7150 2550 2    50   ~ 0
 SCL
-Text Label 7150 2350 2    50   ~ 0
+Text Label 7150 2450 2    50   ~ 0
 SDA
-Text Label 7150 2250 2    50   ~ 0
-MOSI
-Text Label 7150 2150 2    50   ~ 0
-MISO
 $Comp
 L power:+3.3V #PWR0147
 U 1 1 612C22B9
-P 5850 2150
-F 0 "#PWR0147" H 5850 2000 50  0001 C CNN
-F 1 "+3.3V" V 5850 2400 50  0000 C CNN
-F 2 "" H 5850 2150 50  0001 C CNN
-F 3 "" H 5850 2150 50  0001 C CNN
-	1    5850 2150
+P 5850 2550
+F 0 "#PWR0147" H 5850 2400 50  0001 C CNN
+F 1 "+3.3V" V 5850 2800 50  0000 C CNN
+F 2 "" H 5850 2550 50  0001 C CNN
+F 3 "" H 5850 2550 50  0001 C CNN
+	1    5850 2550
 	0    -1   -1   0
 $EndComp
-Text Label 7150 2450 2    50   ~ 0
+Text Label 7150 2350 2    50   ~ 0
 SCK
 $Comp
@@
 	1000 4850 650  4850
 Wire Wire Line
-	650  5050 1000 5050
+	950  5050 1000 5050
 Wire Wire Line
 	650  5250 1000 5250
 Wire Wire Line
-	1400 4850 1750 4850
-Text Label 650  5250 0    50   ~ 0
-SWO
+	1500 4850 1750 4850
 Text Label 650  4650 0    50   ~ 0
 ~RESET
@@
 L power:+3.3V #PWR0151
 U 1 1 613AE3F9
-P 1700 5050
-F 0 "#PWR0151" H 1700 4900 50  0001 C CNN
-F 1 "+3.3V" V 1700 5300 50  0000 C CNN
-F 2 "" H 1700 5050 50  0001 C CNN
-F 3 "" H 1700 5050 50  0001 C CNN
-	1    1700 5050
+P 950 5050
+F 0 "#PWR0151" H 950 4900 50  0001 C CNN
+F 1 "+3.3V" V 950 5300 50  0000 C CNN
+F 2 "" H 950 5050 50  0001 C CNN
+F 3 "" H 950 5050 50  0001 C CNN
+	1    950  5050
 	0    -1   -1   0
 $EndComp
-Wire Wire Line
-	1700 5050 1750 5050
 $Comp
 L power:GND #PWR0152
@@
 Wire Wire Line
 	1000 5450 650  5450
-Wire Wire Line
-	1400 5450 1750 5450
 $Comp
 L Mylib:1_pin_sig J17
@@
 L Mylib:1_pin_sig J20
 U 1 1 61465773
-P 1850 5550
-F 0 "J20" H 1978 5455 50  0000 L CNN
-F 1 "1_pin_sig" H 1978 5410 50  0001 L CNN
-F 2 "Mylib:1.27mm_pin_hole" H 1850 5550 50  0001 C CNN
-F 3 "" H 1850 5550 50  0001 C CNN
-	1    1850 5550
-	1    0    0    -1
+P 5100 5650
+F 0 "J20" H 5228 5555 50  0000 L CNN
+F 1 "1_pin_sig" H 5228 5510 50  0001 L CNN
+F 2 "Mylib:1.27mm_pin_hole" H 5100 5650 50  0001 C CNN
+F 3 "" H 5100 5650 50  0001 C CNN
+	1    5100 5650
+	0    -1   -1   0
 $EndComp
 $Comp
@@
 	1    0    0    -1
 $EndComp
-NoConn ~ 4550 3800
-NoConn ~ 4550 3700
-NoConn ~ 4550 3900
-Wire Wire Line
-	2050 2200 1700 2200
-Text Label 1700 2200 0    50   ~ 0
-D2
 Wire Wire Line
 	650  4650 1000 4650
+Text Label 6500 4000 2    50   ~ 0
+MOSI
+Text Label 6500 3900 2    50   ~ 0
+SCK
+Text Label 6500 4100 2    50   ~ 0
+MISO
 Text Label 6500 3700 2    50   ~ 0
+SCL
+Text Label 6500 3800 2    50   ~ 0
+SDA
+Text Label 4850 4000 0    50   ~ 0
+D5
+Text Label 4850 4100 0    50   ~ 0
+D13
+Text Label 4850 3800 0    50   ~ 0
+D6
+Text Label 4850 3900 0    50   ~ 0
+D12
+Text Label 4850 3700 0    50   ~ 0
+A3
+Text Label 7150 2150 2    50   ~ 0
+MISO
+Wire Wire Line
+	5850 2150 5900 2150
+Text Label 7150 2250 2    50   ~ 0
 MOSI
-Text Label 6500 3800 2    50   ~ 0
-SCK
-Text Label 6500 3900 2    50   ~ 0
-MISO
-Text Label 6500 4000 2    50   ~ 0
-SCL
-Text Label 6500 4100 2    50   ~ 0
-SDA
-Text Label 4850 3700 0    50   ~ 0
+$Comp
+L power:GND #PWR0154
+U 1 1 6187A4E5
+P 5850 2150
+F 0 "#PWR0154" H 5850 1900 50  0001 C CNN
+F 1 "GND" V 5855 2022 50  0000 R CNN
+F 2 "" H 5850 2150 50  0001 C CNN
+F 3 "" H 5850 2150 50  0001 C CNN
+	1    5850 2150
+	0    1    -1   0
+$EndComp
+$Comp
+L power:GND #PWR0155
+U 1 1 6187AE86
+P 6950 1200
+F 0 "#PWR0155" H 6950 950 50  0001 C CNN
+F 1 "GND" V 6955 1072 50  0000 R CNN
+F 2 "" H 6950 1200 50  0001 C CNN
+F 3 "" H 6950 1200 50  0001 C CNN
+	1    6950 1200
+	0    -1   1    0
+$EndComp
+Wire Wire Line
+	650  5650 1000 5650
+Wire Wire Line
+	4250 3800 4550 3800
+Text Label 4550 3700 2    50   ~ 0
+GP0
+Text Label 4550 3800 2    50   ~ 0
+GP1
+Text Label 4550 4000 2    50   ~ 0
+GP3
+Text Label 1500 4650 0    50   ~ 0
+GP0
+Text Label 1700 1400 0    50   ~ 0
+GP2
+Text Label 650  5650 0    50   ~ 0
+GP2
+Wire Wire Line
+	1500 4650 1750 4650
+Wire Wire Line
+	1500 5050 1750 5050
+Wire Wire Line
+	1500 5450 1750 5450
+NoConn ~ 1500 5450
+Wire Wire Line
+	5200 5750 5200 5800
+Text Label 650  5450 0    50   ~ 0
+SWO
+NoConn ~ 1500 4850
+NoConn ~ 1500 5050
+NoConn ~ 650  5250
+NoConn ~ 2050 2200
+Text Label 5650 2350 0    50   ~ 0
+D6
+Text Label 5650 2250 0    50   ~ 0
+D13
+Text Label 7150 1400 2    50   ~ 0
+D6
+Text Label 7150 1300 2    50   ~ 0
+D13
+Text Label 650  4850 0    50   ~ 0
+A5
+$Comp
+L power:GND #PWR0156
+U 1 1 61C6E7D1
+P 10400 4050
+F 0 "#PWR0156" H 10400 3800 50  0001 C CNN
+F 1 "GND" V 10400 3850 50  0000 C CNN
+F 2 "" H 10400 4050 50  0001 C CNN
+F 3 "" H 10400 4050 50  0001 C CNN
+	1    10400 4050
+	0    -1   1    0
+$EndComp
+Text Label 10750 4250 2    50   ~ 0
+MOTOR1_A
+Text Label 10750 4150 2    50   ~ 0
+MOTOR1_B
+$Comp
+L power:VCC #PWR0157
+U 1 1 61D0C464
+P 10400 5550
+F 0 "#PWR0157" H 10400 5400 50  0001 C CNN
+F 1 "VCC" V 10400 5750 50  0000 C CNN
+F 2 "" H 10400 5550 50  0001 C CNN
+F 3 "" H 10400 5550 50  0001 C CNN
+	1    10400 5550
+	0    1    1    0
+$EndComp
+$Comp
+L power:GND #PWR0158
+U 1 1 61D407FD
+P 10400 5250
+F 0 "#PWR0158" H 10400 5000 50  0001 C CNN
+F 1 "GND" V 10400 5050 50  0000 C CNN
+F 2 "" H 10400 5250 50  0001 C CNN
+F 3 "" H 10400 5250 50  0001 C CNN
+	1    10400 5250
+	0    -1   1    0
+$EndComp
+Wire Wire Line
+	10350 5250 10400 5250
+Wire Wire Line
+	10350 4350 10400 4350
+$Comp
+L power:VCC #PWR0159
+U 1 1 61E16D5F
+P 10400 4350
+F 0 "#PWR0159" H 10400 4200 50  0001 C CNN
+F 1 "VCC" V 10400 4550 50  0000 C CNN
+F 2 "" H 10400 4350 50  0001 C CNN
+F 3 "" H 10400 4350 50  0001 C CNN
+	1    10400 4350
+	0    1    1    0
+$EndComp
+Wire Wire Line
+	10350 4050 10400 4050
+Wire Wire Line
+	10350 4450 10750 4450
+Wire Wire Line
+	10350 3950 10750 3950
+Wire Wire Line
+	10400 5550 10350 5550
+Wire Wire Line
+	10350 5150 10750 5150
+Wire Wire Line
+	10350 5650 10750 5650
+Text Label 10750 4450 2    50   ~ 0
+M1_O1
+Text Label 10750 3950 2    50   ~ 0
+M1_O2
+Text Label 10750 5650 2    50   ~ 0
+M2_O1
+Text Label 10750 5150 2    50   ~ 0
+M2_O2
+Text Label 1700 4100 0    50   ~ 0
+MOTOR1_A
+Text Label 1700 4300 0    50   ~ 0
+MOTOR1_B
+Text Label 10750 5450 2    50   ~ 0
 D5
-Text Label 4850 3800 0    50   ~ 0
+Text Label 10750 5350 2    50   ~ 0
 D13
-Text Label 4850 3900 0    50   ~ 0
-D11
-Text Label 4850 4000 0    50   ~ 0
-D6
-Text Label 4850 4100 0    50   ~ 0
-D12
+NoConn ~ 10100 2350
 $EndSCHEMATC
