File: PCB/Mainboard/V1/mainboard_v1/mainboard_v1.kicad_pcb (KiCad board)
At the start: 2 copper layers, 35 x 40 mm, 44 parts, among them J1 22-23-2021, J2 USB_B_Micro, J5 M50-3100545, J6 M50-3100545, J7 M50-3100545, SW1 SW_SPDT, U1 MDBT50Q-1MV2, U3 MCP73831T-2ACI_OT, U4 AP2112K-3.3, U5 MPU6050

Commit message: udated by FZ
Parts:
- removed H4: M2, Mylib:mounthole_1.8mm
- removed H5, H6: M2, Mylib:M2_NPTH_mounting_hole
- added C14: 10uF, Capacitor_SMD:C_0603_1608Metric_Pad1.08x0.95mm_HandSolder, F.Cu at (191.0, 108.1)
- added C15: 10uF, Capacitor_SMD:C_0603_1608Metric_Pad1.08x0.95mm_HandSolder, F.Cu at (197.4, 107.2)
- added C16: 10uF, Capacitor_SMD:C_0603_1608Metric_Pad1.08x0.95mm_HandSolder, F.Cu at (197.7, 113.7)
- added C17: 10uF, Capacitor_SMD:C_0603_1608Metric_Pad1.08x0.95mm_HandSolder, F.Cu at (193.6, 119.8)
- added C18: 0.1uF, Capacitor_SMD:C_0603_1608Metric_Pad1.08x0.95mm_HandSolder, F.Cu at (192.9, 122.5)
- added IC1: MP6513GJ-Z, SamacSys_Parts:SOT95P280X100-6N, F.Cu at (178.5, 103.5)
- added IC2: MP6513GJ-Z, SamacSys_Parts:SOT95P280X100-6N, F.Cu at (201.3, 119.0)
- added J10: 1_pin_sig, Mylib:1.27mm_pin_hole, F.Cu at (184.8, 129.6)
- added J11: 1_pin_sig, Mylib:1.27mm_pin_hole, F.Cu at (185.5, 126.6)
- added J12: 1_pin_sig, Mylib:1.27mm_pin_hole, F.Cu at (183.3, 129.6)
- added J13: 1_pin_sig, Mylib:1.27mm_pin_hole, F.Cu at (186.5, 128.1)
- added J14: 1_pin_sig, Mylib:1.27mm_pin_hole, F.Cu at (189.5, 128.1)
- added J15: 1_pin_sig, Mylib:1.27mm_pin_hole, F.Cu at (183.3, 126.6)
- added J16: 1_pin_sig, Mylib:1.27mm_pin_hole, F.Cu at (188.0, 128.1)
- added J17: 1_pin_sig, Mylib:1.27mm_pin_hole, F.Cu at (178.8, 125.1)
- added J18: 1_pin_sig, Mylib:1.27mm_pin_hole, F.Cu at (180.3, 126.6)
- added J19: 1_pin_sig, Mylib:1.27mm_pin_hole, F.Cu at (180.3, 125.1)
- added J20: 1_pin_sig, Mylib:1.27mm_pin_hole, F.Cu at (181.8, 125.1)
- added J3: 1734592-6, SamacSys_Parts:17345926, B.Cu at (178.4, 100.6)
- added J4: 22-23-2021, Connector_PinHeader_1.27mm:PinHeader_2x01_P1.27mm_Vertical, F.Cu at (195.0, 96.1)
- added J8: 1734592-6, SamacSys_Parts:17345926, B.Cu at (201.6, 118.2)
- added J9: 1_pin_sig, Mylib:1.27mm_pin_hole, F.Cu at (181.1, 126.6)
- added R10: 10k, Resistor_SMD:R_0603_1608Metric_Pad0.98x0.95mm_HandSolder, B.Cu at (193.4, 98.9)
- added R11: 10k, Resistor_SMD:R_0603_1608Metric_Pad0.98x0.95mm_HandSolder, B.Cu at (191.9, 98.9)
- added S1: B3U-1000P, digikey-footprints:Switch_Tactile_SMD_B3U-1000P, F.Cu at (178.9, 97.7)
- added U7: AP2112K-3.3, Package_TO_SOT_SMD:SOT-23-5_HandSoldering, F.Cu at (195.4, 122.8)
- C10, C11, R1, R2, R5, R7, U3, U4: moved to F.Cu
- C12, C8: value 10uF -> 0.1uF
- C13: value 10uF -> TAJP106K010RNJ; footprint Capacitor_SMD:C_0603_1608Metric_Pad1.08x0.95mm_HandSolder -> SamacSys_Parts:CAPPM2014X170N; moved to B.Cu
- C2: value 0.1uF -> 10uF
- C9: value 10uF -> TAJP106K010RNJ; footprint Capacitor_SMD:C_0603_1608Metric_Pad1.08x0.95mm_HandSolder -> SamacSys_Parts:CAPPM2014X170N; moved to F.Cu
- J5, J7: value M50-3100545 -> 20021321-00010C4LF
- J6: value M50-3100545 -> 20021321-00014C1LF; footprint SnapEDA Library:HARWIN_M50-3100545 -> SamacSys_Parts:2002132100014C1LF
- R6: value 10k -> 4.99k; moved to F.Cu
- R8, R9, SW1: moved to B.Cu
- XTAL1: footprint digikey-footprints:SMD-2_3.2x1.5mm -> SamacSys_Parts:ECS32712512TR
- moved H1 107.1 mm to (190.0, 123.0)
- moved H3 94.4 mm to (201.8, 108.0)
- moved R2 84.2 mm to (185.2, 109.8), turned to 0 degrees
- moved R1 83.8 mm to (185.2, 111.3), turned to 180 degrees
- moved J5 83.5 mm to (190.0, 127.8)
- moved R3 82.2 mm to (181.6, 111.0), turned to 0 degrees
- moved R4 81.8 mm to (181.6, 112.7), turned to 0 degrees
- moved L1 80.6 mm to (192.5, 108.1)
- moved C11 80.2 mm to (182.4, 122.5), turned to 270 degrees
- moved D4 80.2 mm to (202.3, 112.2), turned to 90 degrees
- moved C2 79.5 mm to (189.4, 108.1)
- moved U1 79.2 mm to (187.7, 98.0)
- moved C1 78.9 mm to (198.8, 97.8)
- moved U5 78.9 mm to (198.4, 101.5)
- moved C3 78.9 mm to (202.0, 103.8)
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Connections:
- C12 pad 2: +3V3 -> VCC
- C13 pad 1: GND -> VBUS
- C13 pad 2: Net-(C11-Pad2) -> GND
- C8 pad 2: +3V3 -> VCC
- C9 pad 1: GND -> Net-(C11-Pad2)
- C9 pad 2: VBUS -> GND
- J5 pad 1: (no net) -> /SCL
- J5 pad 10: (no net) -> +3V3
- J5 pad 2: (no net) -> /A1
- J5 pad 3: (no net) -> /SCK
- J5 pad 5: (no net) -> /SDA
- J5 pad 7: (no net) -> /MOSI
- J5 pad 9: (no net) -> /MISO
- J6 pad 1: (no net) -> GND
- J6 pad 10: (no net) -> /D13
- J6 pad 2: (no net) -> VPP
- J6 pad 3: (no net) -> /SDA
- J6 pad 4: (no net) -> /D12
- J6 pad 5: (no net) -> /SCL
- J6 pad 6: (no net) -> /D6
- J6 pad 7: (no net) -> /MISO
- J6 pad 8: (no net) -> /D11
- J6 pad 9: (no net) -> /SCK
- J7 pad 1: (no net) -> +3V3
- J7 pad 10: (no net) -> /SCL
- J7 pad 2: (no net) -> /MISO
- J7 pad 4: (no net) -> /MOSI
- J7 pad 6: (no net) -> /SDA
- J7 pad 8: (no net) -> /SCK
- J7 pad 9: (no net) -> /A1
- L1 pad 1: (no net) -> +3V3
- R1 pad 1: /ADC_BAT -> /A0
- R2 pad 2: /ADC_BAT -> /A0
- SW1 pad 1: VPP -> (no net)
- SW1 pad 2: Net-(C11-Pad2) -> VPP
- SW1 pad 3: (no net) -> Net-(C11-Pad2)
- U1 pad 10: (no net) -> /M1_IN2
- U1 pad 12: /ADC_BAT -> (no net)
- U1 pad 14: (no net) -> /LED1
- U1 pad 16: (no net) -> /LED2
- U1 pad 20: (no net) -> /A0
- U1 pad 21: (no net) -> /A1
- U1 pad 22: (no net) -> /D11
- U1 pad 23: (no net) -> /D6
- U1 pad 24: (no net) -> /D12
- U1 pad 25: (no net) -> /D5
- U1 pad 26: (no net) -> /D13
- U1 pad 27: (no net) -> /SCL
- U1 pad 29: (no net) -> /SDA
- U1 pad 36: /SCL -> /SCK
- U1 pad 37: (no net) -> /MOSI
- U1 pad 38: /SDA -> (no net)
- U1 pad 39: (no net) -> /MISO
- U1 pad 40: (no net) -> /~RESET
- U1 pad 47: /LED1 -> /SWO
- U1 pad 51: (no net) -> /SWDIO
- U1 pad 53: (no net) -> /SWDCLK
- U1 pad 61: /LED2 -> (no net)
- U1 pad 8: (no net) -> /M1_IN1
Routing:
- net +3V3: track 2.55 -> 66.2 mm, vias 0 -> 4
- net /~RESET: track 0.00 -> 42.5 mm, vias 0 -> 1
- net VCC: track 0.00 -> 42.0 mm, vias 0 -> 2
- net Net-(C11-Pad2): track 2.18 -> 43.2 mm, vias 0 -> 2
- net VPP: track 0.00 -> 32.4 mm, vias 0 -> 1
- net VBUS: track 0.00 -> 30.6 mm, vias 0 -> 3
- net /SDA: track 10.6 -> 0.00 mm, vias 2 -> 0
- net /LED1: track 0.00 -> 10.1 mm, vias 0 -> 2
- net GND: track 0.00 -> 9.69 mm, vias 0 -> 4
- net /LED2: track 0.00 -> 8.74 mm, vias 0 -> 2
- net /SCL: track 8.18 -> 0.00 mm, vias 2 -> 0
- net /A0: track 0.00 -> 6.91 mm
- net Net-(R7-Pad2): track 0.00 -> 5.72 mm
- net /SWDIO: track 0.00 -> 5.02 mm
- net /M1_O2: track 0.00 -> 4.92 mm, vias 0 -> 1
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Other:
- board size 35 x 40 mm -> 28 x 41 mm
- copper layers 2 -> 4
- board text added: "+"
- board text added: "@MIT Media Lab SEI"
- board text added: "OFF"
- board text added: "ON"
- board text added: "SWDCLK"
- board text added: "SWDIO"
- board text removed: "MIT Media Lab Space Exploration Initiative"

Commit message: udated by FZ
Parts:
- moved R11 6.61 mm to (195.6, 104.4), turned to 0 degrees
- moved J3 2.60 mm to (178.4, 98.0)
- moved R10 1.23 mm to (192.6, 99.9)
- moved IC2 1.05 mm to (201.2, 120.0)
- moved C8 1.05 mm to (198.2, 119.1)
- moved S1 0.33 mm to (178.9, 97.4)
- moved J17 0.30 mm to (178.5, 125.1)
- moved C15 0.21 mm to (197.6, 107.2)
- moved J18 0.20 mm to (180.1, 126.6)
- moved J19 0.20 mm to (180.1, 125.1)
- moved J8 0.19 mm to (201.6, 118.0)
- moved J14 0.10 mm to (189.6, 128.1)
- moved J10 0.10 mm to (184.9, 129.6)
- moved J11 0.10 mm to (185.6, 126.6)
- moved J13 0.10 mm to (186.4, 128.1)
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Connections:
- D3 pad 1: Net-(D3-Pad1) -> GND
- D3 pad 2: Net-(C11-Pad2) -> Net-(D3-Pad2)
- IC1 pad 4: (no net) -> /M1_O2
- IC1 pad 6: (no net) -> /M1_O1
- IC2 pad 4: (no net) -> /M2_O2
- IC2 pad 6: (no net) -> /M2_O1
- J11 pad 1: (no net) -> +3V3
- J12 pad 1: +3V3 -> (no net)
- J13 pad 1: /SWO -> (no net)
- J15 pad 1: (no net) -> /SWO
- J18 pad 1: (no net) -> /GP0
- J19 pad 1: (no net) -> /GP2
- J20 pad 1: (no net) -> Net-(C11-Pad2)
- J3 pad 1: (no net) -> /M1_O2
- J3 pad 2: (no net) -> GND
- J3 pad 3: (no net) -> /MOTOR1_B
- J3 pad 4: (no net) -> /MOTOR1_A
- J3 pad 5: (no net) -> VCC
- J3 pad 6: (no net) -> /M1_O1
- J5 pad 1: /SCL -> /MISO
- J5 pad 2: /A1 -> GND
- J5 pad 3: /SCK -> /MOSI
- J5 pad 4: (no net) -> /D13
- J5 pad 5: /SDA -> /SCK
- J5 pad 6: (no net) -> /D6
- J5 pad 7: /MOSI -> /SDA
- J5 pad 8: (no net) -> /A1
- J5 pad 9: /MISO -> /SCL
- J6 pad 10: /D13 -> /D6
- J6 pad 11: /MOSI -> /SCL
- J6 pad 12: /D5 -> /A3
- J6 pad 3: /SDA -> /MISO
- J6 pad 4: /D12 -> /D13
- J6 pad 5: /SCL -> /MOSI
- J6 pad 6: /D6 -> /D5
- J6 pad 7: /MISO -> /SCK
- J6 pad 8: /D11 -> /D12
- J6 pad 9: /SCK -> /SDA
- J7 pad 1: +3V3 -> GND
- J7 pad 3: (no net) -> /D13
- J7 pad 5: (no net) -> /D6
- J7 pad 6: /SDA -> /SCK
- J7 pad 7: (no net) -> /A1
- J7 pad 8: /SCK -> /SDA
- J7 pad 9: /A1 -> +3V3
- J8 pad 1: (no net) -> /M2_O2
- J8 pad 2: (no net) -> GND
- J8 pad 3: (no net) -> /D13
- J8 pad 4: (no net) -> /D5
- J8 pad 5: (no net) -> VCC
- J8 pad 6: (no net) -> /M2_O1
- J9 pad 1: (no net) -> /A5
- R5 pad 1: Net-(D3-Pad1) -> Net-(C11-Pad2)
- R5 pad 2: GND -> Net-(D3-Pad2)
- U1 pad 10: /M1_IN2 -> /MOTOR1_A
- U1 pad 11: (no net) -> /GP2
- U1 pad 12: (no net) -> /MOTOR1_B
- U1 pad 13: (no net) -> /A3
- U1 pad 22: /D11 -> (no net)
- U1 pad 4: (no net) -> /GP0
- U1 pad 6: (no net) -> /M1_IN1
- U1 pad 8: /M1_IN1 -> /M1_IN2
- U1 pad 9: (no net) -> /A5
- U5 pad 19: Net-(U5-Pad19) -> (no net)
- U5 pad 21: Net-(U5-Pad19) -> (no net)
Routing:
- net /SCL: track 0.00 -> 39.2 mm, vias 0 -> 5
- net /SDA: track 0.00 -> 36.9 mm, vias 0 -> 5
- net /SWO: track 0.00 -> 34.3 mm, vias 0 -> 1
- net /GP0: track 0.00 -> 33.0 mm, vias 0 -> 1
- net /D13: track 0.00 -> 30.7 mm, vias 0 -> 4
- net /A5: track 0.00 -> 30.5 mm, vias 0 -> 1
- net /MISO: track 1.45 -> 30.9 mm, vias 1 -> 4
- net /D5: track 0.00 -> 29.1 mm, vias 0 -> 2
- net /MOSI: track 1.15 -> 29.6 mm, vias 1 -> 4
- net /SCK: track 1.05 -> 29.3 mm, vias 1 -> 4
- net /GP2: track 0.00 -> 27.8 mm, vias 0 -> 1
- net /D6: track 0.00 -> 26.8 mm, vias 0 -> 3
- net /A1: track 0.84 -> 26.4 mm, vias 1 -> 2
- net /A3: track 0.00 -> 17.4 mm, vias 0 -> 2
- net +3V3: track 66.2 -> 83.0 mm, vias 4 -> 5
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- added copper zone on B.Cu, net GND
- added copper zone on F.Cu, net GND
- added copper zone on GND, net GND
- added copper zone on PWR, net GND

Commit message: udated by FZ
Connections:
- IC2 pad 1: (no net) -> /M2_IN1
- IC2 pad 3: (no net) -> /M2_IN2
- J5 pad 4: /D13 -> /D11
- J6 pad 4: /D13 -> /D11
- J6 pad 6: /D5 -> /D9
- J7 pad 3: /D13 -> /D11
- U1 pad 19: (no net) -> /D9
- U1 pad 22: (no net) -> /D11
- U1 pad 44: (no net) -> /M2_IN1
- U1 pad 46: (no net) -> /M2_IN2
Routing:
- net /M2_IN1: track 0.00 -> 27.3 mm, vias 0 -> 2
- net /D11: track 0.00 -> 27.1 mm, vias 0 -> 4
- net /M2_IN2: track 0.00 -> 25.7 mm, vias 0 -> 2
- net /D9: track 0.00 -> 19.4 mm, vias 0 -> 2
- net /D13: track 30.7 -> 22.5 mm, vias 4 -> 1
- net /D5: track 29.1 -> 28.0 mm, vias 2 -> 1
- net /SCL: track 39.2 -> 39.9 mm
- net /M2_O1: track 4.98 -> 5.55 mm
- net /A0: track 6.91 -> 6.83 mm, vias 0 -> 2
- net GND: vias 53 -> 60
