File: PCB/IR_TEMP_module/IR_TEMP_V2/IR_TEMP_V1.kicad_pcb (KiCad board)
At the start: 2 copper layers, 10 x 20 mm, 26 parts, among them IC1 LMP91051MTX_NOPB, J1 1_PIN, J10 1_PIN, J11 1_PIN, J12 1_PIN, J2 1_PIN, J3 1_PIN, J4 1_PIN, J5 1_PIN, J6 1_PIN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

Commit message: udated by FZ
Parts:
- removed C3, C4: 0.01uF, Capacitor_SMD:C_0402_1005Metric_Pad0.74x0.62mm_HandSolder
- removed C5: 1uF, Capacitor_SMD:C_0402_1005Metric_Pad0.74x0.62mm_HandSolder
- removed C6: 6800pF, Capacitor_SMD:C_0402_1005Metric_Pad0.74x0.62mm_HandSolder
- removed IC1: LMP91051MTX_NOPB, SamacSys_Parts:SOP65P640X120-14N
- R2, R3: value 160k -> 100k
- U1: value ZTP-135SR -> TPIS_1T_1084; footprint Mylib:TO-46-4 -> Mylib:TPIS_1T_1084; moved to F.Cu
- moved C1 8.55 mm to (116.3, 70.5), turned to 270 degrees
- moved J1 8.04 mm to (114.8, 69.9)
- moved J7 8.04 mm to (114.8, 73.9)
- moved J10 5.70 mm to (112.7, 73.9)
- moved J4 5.70 mm to (112.7, 69.9)
- moved R2 5.32 mm to (116.8, 67.9), turned to 270 degrees
- moved J2 5.27 mm to (114.8, 68.5)
- moved J8 5.27 mm to (114.8, 72.5)
- moved R3 5.22 mm to (114.8, 64.7), turned to 225 degrees
- moved R1 5.02 mm to (112.5, 67.9), turned to 270 degrees
- moved C2 4.65 mm to (113.4, 63.6), turned to 180 degrees
- moved J3 3.46 mm to (112.7, 68.5)
- moved J9 3.46 mm to (112.7, 72.6)
- moved J11 0.90 mm to (110.4, 72.5)
- moved J12 0.90 mm to (110.4, 73.9)
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Connections:
- J10 pad 1: /Temp_A -> /SCL
- J11 pad 1: /SCLK -> /A1
- J12 pad 1: /MOSI -> /INT
- J3 pad 1: /SPICS -> /SDA
- J4 pad 1: /Temp_A -> /SCL
- J5 pad 1: /SCLK -> /A1
- J6 pad 1: /MOSI -> /INT
- J9 pad 1: /SPICS -> /SDA
- R1 pad 1: +3V3 -> /SDA
- R1 pad 2: /Thermistor -> +3V3
- R2 pad 1: /Temp_A -> /SCL
- R2 pad 2: Net-(IC1-Pad9) -> +3V3
- R3 pad 1: /A1 -> /INT_TPIS
- R3 pad 2: /A0 -> /INT
- U1 pad 2: Net-(C3-Pad2) -> +3V3
- U1 pad 3: /Thermistor -> /SDA
- U1 pad 4: /CMOUT -> /INT_TPIS
Routing:
- net /MOSI: track 14.7 -> 0.00 mm, vias 2 -> 0
- net /SCLK: track 14.2 -> 0.00 mm, vias 2 -> 0
- net /SPICS: track 13.7 -> 0.00 mm, vias 2 -> 0
- net +3V3: track 6.65 -> 17.9 mm, vias 1 -> 2
- net Net-(IC1-Pad9): track 11.2 -> 0.00 mm
- net /INT: track 0.00 -> 10.3 mm, vias 0 -> 1
- net /SCL: track 0.00 -> 9.55 mm, vias 0 -> 1
- net Net-(C3-Pad2): track 7.73 -> 0.00 mm
- net /CMOUT: track 7.66 -> 0.00 mm, vias 1 -> 0
- net /SDA: track 0.00 -> 6.49 mm, vias 0 -> 1
- net /A1: track 3.36 -> 7.76 mm
- net /A0: track 3.58 -> 0.00 mm, vias 1 -> 0
- net /Temp_A: track 2.81 -> 0.00 mm, vias 1 -> 0
- net /INT_TPIS: track 0.00 -> 2.19 mm
- net GND: track 1.62 -> 0.00 mm, vias 21 -> 13
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Other:
- board text added: "AstroAnt IR"

Commit message: udated by FZ
Parts:
- moved R3 6.37 mm to (109.7, 68.6), turned to 270 degrees
Routing:
- net /INT_TPIS: track 2.19 -> 9.19 mm
- net /INT: track 10.3 -> 3.54 mm
Changed lines of the file:
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@@
   )
   (module Resistor_SMD:R_0402_1005Metric_Pad0.72x0.64mm_HandSolder (layer B.Cu)
-    (at 114.77 64.68 225)
+    (at 109.72 68.56 270)
     (descr "Resistor SMD 0402 (1005 Metric), square (rectangular) end terminal, IPC_7351 nominal with elongated pad for handsoldering. (Body size source: IPC-SM-782 page 72, https://www.pcb-3d.com/wordpress/wp-content/uploads/ipc-sm-782a_amendment_1_and_2.pdf), generated with kicad-footprint-generator")
     (tags "resistor handsolder")
     (attr smd)
-    (fp_text reference R3 (at 0 1.17 45) (layer B.SilkS) hide
-      (effects (font (size 1 1) (thickness 0.15)) (justify mirror))
-    )
-    (fp_text value 100k (at 0 -1.17 45) (layer B.Fab)
-      (effects (font (size 1 1) (thickness 0.15)) (justify mirror))
-    )
-    (fp_text user %R (at 0 0 45) (layer B.Fab)
+    (fp_text reference R3 (at 0 1.17 90) (layer B.SilkS) hide
+      (effects (font (size 1 1) (thickness 0.15)) (justify mirror))
+    )
+    (fp_text value 100k (at 0 -1.17 90) (layer B.Fab)
+      (effects (font (size 1 1) (thickness 0.15)) (justify mirror))
+    )
+    (fp_text user %R (at 0 0 90) (layer B.Fab)
       (effects (font (size 0.26 0.26) (thickness 0.04)) (justify mirror))
     )
@@
     (fp_line (start 1.1 0.47) (end 1.1 -0.47) (layer B.CrtYd) (width 0.05))
     (fp_line (start 1.1 -0.47) (end -1.1 -0.47) (layer B.CrtYd) (width 0.05))
-    (pad 2 smd roundrect (at 0.5975 0 225) (size 0.715 0.64) (layers B.Cu B.Paste B.Mask) (roundrect_rratio 0.25)
+    (pad 2 smd roundrect (at 0.5975 0 270) (size 0.715 0.64) (layers B.Cu B.Paste B.Mask) (roundrect_rratio 0.25)
       (net 6 /INT))
-    (pad 1 smd roundrect (at -0.5975 0 225) (size 0.715 0.64) (layers B.Cu B.Paste B.Mask) (roundrect_rratio 0.25)
+    (pad 1 smd roundrect (at -0.5975 0 270) (size 0.715 0.64) (layers B.Cu B.Paste B.Mask) (roundrect_rratio 0.25)
       (net 7 /INT_TPIS))
     (model ${KISYS3DMOD}/Resistor_SMD.3dshapes/R_0402_1005Metric.wrl
@@
   (via (at 115.75 73.16) (size 0.508) (drill 0.3048) (layers F.Cu B.Cu) (net 2))
   (via (at 111.28 73.16) (size 0.508) (drill 0.3048) (layers F.Cu B.Cu) (net 2))
-  (segment (start 115.16757 66.548053) (end 112.061947 66.548053) (width 0.1524) (layer B.Cu) (net 3))
-  (segment (start 110.4 68.21) (end 110.4 70.512) (width 0.1524) (layer B.Cu) (net 3))
+  (segment (start 115.16757 66.548053) (end 111.565513 66.548053) (width 0.1524) (layer B.Cu) (net 3))
+  (segment (start 110.4 67.713566) (end 110.4 70.512) (width 0.1524) (layer B.Cu) (net 3))
+  (segment (start 111.565513 66.548053) (end 110.4 67.713566) (width 0.1524) (layer B.Cu) (net 3))
+  (segment (start 110.4 70.512) (end 110.4 70.512) (width 0.1524) (layer B.Cu) (net 3))
   (via (at 110.4 70.512) (size 0.508) (drill 0.3048) (layers F.Cu B.Cu) (net 3))
-  (segment (start 112.061947 66.548053) (end 110.4 68.21) (width 0.1524) (layer B.Cu) (net 3))
   (segment (start 112.65 70.468) (end 112.65 70.468) (width 0.1524) (layer F.Cu) (net 4))
   (segment (start 111.90139 67.85111) (end 112.45 67.3025) (width 0.1524) (layer F.Cu) (net 4))
@@
   (segment (start 116.747728 67.300228) (end 116.75 67.3025) (width 0.1524) (layer F.Cu) (net 5))
   (segment (start 116.747728 64.967436) (end 116.747728 67.300228) (width 0.1524) (layer F.Cu) (net 5))
-  (segment (start 114.347504 65.102496) (end 113.206757 66.243243) (width 0.1524) (layer B.Cu) (net 6))
-  (segment (start 111.93569 66.243244) (end 109.33 68.848934) (width 0.1524) (layer B.Cu) (net 6))
-  (segment (start 113.206757 66.243243) (end 111.93569 66.243244) (width 0.1524) (layer B.Cu) (net 6))
+  (segment (start 109.72 69.1575) (end 109.34 69.5375) (width 0.1524) (layer B.Cu) (net 6))
   (segment (start 110.4 71.936) (end 110.4 71.936) (width 0.1524) (layer B.Cu) (net 6))
-  (segment (start 109.33 71.17) (end 109.33 68.848934) (width 0.1524) (layer B.Cu) (net 6))
-  (segment (start 110.096 71.936) (end 109.33 71.17) (width 0.1524) (layer B.Cu) (net 6))
-  (segment (start 110.4 71.936) (end 110.096 71.936) (width 0.1524) (layer B.Cu) (net 6))
+  (segment (start 109.34 71.15) (end 109.34 69.5375) (width 0.1524) (layer B.Cu) (net 6))
+  (segment (start 110.126 71.936) (end 109.34 71.15) (width 0.1524) (layer B.Cu) (net 6))
+  (segment (start 110.4 71.936) (end 110.126 71.936) (width 0.1524) (layer B.Cu) (net 6))
   (via (at 110.4 71.936) (size 0.508) (drill 0.3048) (layers F.Cu B.Cu) (net 6))
-  (segment (start 115.222979 64.257504) (end 115.192496 64.257504) (width 0.1524) (layer B.Cu) (net 7))
-  (segment (start 116.748053 62.73243) (end 115.222979 64.257504) (width 0.1524) (layer B.Cu) (net 7))
+  (segment (start 116.748053 62.73243) (end 113.23724 66.243243) (width 0.1524) (layer B.Cu) (net 7))
+  (segment (start 111.439257 66.243243) (end 109.72 67.9625) (width 0.1524) (layer B.Cu) (net 7))
+  (segment (start 113.23724 66.243243) (end 111.439257 66.243243) (width 0.1524) (layer B.Cu) (net 7))
   (zone (net 2) (net_name GND) (layer F.Cu) (hatch edge 0.508)
     (connect_pads (clearance 0.1524))
