File: PCB/IR_TEMP_module/IR_TEMP_V2/IR_TEMP_V1.sch (KiCad schematic (older format))
At the start: 26 parts, among them IC1 LMP91051MTX_NOPB, J1 1_PIN, J10 1_PIN, J11 1_PIN, J12 1_PIN, J2 1_PIN, J3 1_PIN, J4 1_PIN, J5 1_PIN, J6 1_PIN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

Commit message: udated by FZ
Parts:
- removed C3, C4: 0.01uF, Capacitor_SMD:C_0402_1005Metric_Pad0.74x0.62mm_HandSolder, symbol Device:C_Small
- removed C5: 1uF, Capacitor_SMD:C_0402_1005Metric_Pad0.74x0.62mm_HandSolder, symbol Device:C_Small
- removed C6: 6800pF, Capacitor_SMD:C_0402_1005Metric_Pad0.74x0.62mm_HandSolder, symbol Device:C_Small
- removed IC1: LMP91051MTX_NOPB, SamacSys_Parts:SOP65P640X120-14N, symbol SamacSys_Parts:LMP91051MTX_NOPB
- removed R3: 160k, Resistor_SMD:R_0402_1005Metric_Pad0.72x0.64mm_HandSolder, symbol Device:R_Small
- removed U1: ZTP-135SR, Mylib:TO-46-4, symbol SamacSys_Parts:ZTP-135SR
- added R?: 100k, Resistor_SMD:R_0402_1005Metric_Pad0.72x0.64mm_HandSolder, symbol Device:R_Small
- added U1: TPIS_1T_1084, Mylib:TPIS_1T_1084, symbol Mylib:TPIS_1T_1084
- R2: value 160k -> 100k
Connections:
- net SCLK is gone; now on net A1: J11.1, J5.1
- net Thermistor is gone; now on net +3V3: R1.2
- net +3V3: now also R2.2, U1.2 (VDD); no longer R1.1
- net A1: now also U1.6 (A1)
- net GND: now also U1.1 (GND)
- net MOSI renamed INT
- net INT: now also R?.2
- net SPICS renamed SDA
- net SDA: now also R1.1, U1.3 (SDA)
- net Temp_A renamed SCL
- net SCL: now also U1.5 (SCL)
- new net INT_TPIS: R?.1, U1.4 (INT)
- no-connect marks 3 -> 0
Other:
- moved on the sheet: C1, C2

Commit message: udated by FZ
Parts:
- R1, R2: value 100k -> 10k
- R3: renamed from R?; value 100k -> 10k
Changed lines of the file:
@@
 P 4400 4500
 F 0 "R1" V 4330 4500 50  0000 C CNN
-F 1 "100k" V 4470 4500 50  0000 C CNN
+F 1 "10k" V 4470 4500 50  0000 C CNN
 F 2 "Resistor_SMD:R_0402_1005Metric_Pad0.72x0.64mm_HandSolder" H 4400 4500 50  0001 C CNN
 F 3 "~" H 4400 4500 50  0001 C CNN
@@
 P 4400 4750
 F 0 "R2" V 4330 4750 50  0000 C CNN
-F 1 "100k" V 4470 4750 50  0000 C CNN
+F 1 "10k" V 4470 4750 50  0000 C CNN
 F 2 "Resistor_SMD:R_0402_1005Metric_Pad0.72x0.64mm_HandSolder" H 4400 4750 50  0001 C CNN
 F 3 "~" H 4400 4750 50  0001 C CNN
@@
 A1
 $Comp
-L Device:R_Small R?
+L Device:R_Small R3
 U 1 1 61619CEE
 P 4400 5050
-F 0 "R?" V 4330 5050 50  0000 C CNN
-F 1 "100k" V 4470 5050 50  0000 C CNN
+F 0 "R3" V 4330 5050 50  0000 C CNN
+F 1 "10k" V 4470 5050 50  0000 C CNN
 F 2 "Resistor_SMD:R_0402_1005Metric_Pad0.72x0.64mm_HandSolder" H 4400 5050 50  0001 C CNN
 F 3 "~" H 4400 5050 50  0001 C CNN
