File: PCB/Mainboard/mainboard_v1/mainboard_v1.sch (KiCad schematic (older format))
At the start: 67 parts, among them IC1 MP6513GJ-Z, IC2 MP6513GJ-Z, J1 22-23-2021, J10 1_pin_sig, J11 1_pin_sig, J12 1_pin_sig, J13 1_pin_sig, J14 1_pin_sig, J15 1_pin_sig, J16 1_pin_sig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

Commit message: udated by FZ
Parts:
- R1, R2: value 100k -> 49.9k
- R3, R4: value 1k -> 4.99k
Changed lines of the file:
@@
 P 2800 4850
 F 0 "R1" V 2700 4850 50  0000 C CNN
-F 1 "100k" V 2900 4850 50  0000 C CNN
+F 1 "49.9k" V 2900 4850 50  0000 C CNN
 F 2 "Resistor_SMD:R_0603_1608Metric_Pad0.98x0.95mm_HandSolder" H 2800 4850 50  0001 C CNN
 F 3 "~" H 2800 4850 50  0001 C CNN
@@
 P 3400 4850
 F 0 "R2" V 3300 4850 50  0000 C CNN
-F 1 "100k" V 3500 4850 50  0000 C CNN
+F 1 "49.9k" V 3500 4850 50  0000 C CNN
 F 2 "Resistor_SMD:R_0603_1608Metric_Pad0.98x0.95mm_HandSolder" H 3400 4850 50  0001 C CNN
 F 3 "~" H 3400 4850 50  0001 C CNN
@@
 P 2900 5200
 F 0 "R3" V 2800 5200 50  0000 C CNN
-F 1 "1k" V 3000 5200 50  0000 C CNN
+F 1 "4.99k" V 3000 5200 50  0000 C CNN
 F 2 "Resistor_SMD:R_0603_1608Metric_Pad0.98x0.95mm_HandSolder" H 2900 5200 50  0001 C CNN
 F 3 "~" H 2900 5200 50  0001 C CNN
@@
 P 2900 5550
 F 0 "R4" V 2800 5550 50  0000 C CNN
-F 1 "1k" V 3000 5550 50  0000 C CNN
+F 1 "4.99k" V 3000 5550 50  0000 C CNN
 F 2 "Resistor_SMD:R_0603_1608Metric_Pad0.98x0.95mm_HandSolder" H 2900 5550 50  0001 C CNN
 F 3 "~" H 2900 5550 50  0001 C CNN
