File: PCB/Mainboard/mainboard_v1/mainboard_v1.kicad_pcb (KiCad board)
At the start: 4 copper layers, 28 x 41 mm, 67 parts, among them IC1 MP6513GJ-Z, IC2 MP6513GJ-Z, J1 22-23-2021, J10 1_pin_sig, J11 1_pin_sig, J12 1_pin_sig, J13 1_pin_sig, J14 1_pin_sig, J15 1_pin_sig, J16 1_pin_sig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

Commit message: udated by FZ
Parts:
- D1: value LED -> LED_white
- D2: value LED -> LED_red
- R1, R2: value 100k -> 49.9k
- R3, R4, R5: value 1k -> 4.99k

Commit message: udated by FZ
Connections:
- net /~RESET renamed /~{RESET}
Routing:
- net GND: track 13.3 -> 11.6 mm
- added copper zone on In1.Cu, net GND
- added copper zone on In2.Cu, net GND
- removed copper zone on GND, net GND
- removed copper zone on PWR, net GND
Other:
- net class Default removed
