File: PCB/Camera/Camera.kicad_pcb (KiCad board)
At the start: 2 copper layers, 24 x 19 mm, 4 parts, among them J1 GRPB052VWVN-RC, J2 GRPB052VWVN-RC, U1 Arducam_OV2640_module

Commit message: udated by FZ
Parts:
- moved J2 0.96 mm to (152.0, 83.5)
Changed lines of the file:
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@@
   )
   (module SamacSys_Parts:HDRV10W50P127_2X5_635X340X430P (layer F.Cu)
-    (at 152 82.55)
+    (at 152.01 83.505)
     (descr GRPB052VWVN-RC)
     (tags Connector)
@@
       (effects (font (size 1.27 1.27) (thickness 0.254)))
     )
+    (fp_line (start 3.44 -1.85) (end -2.54 -1.85) (layer F.SilkS) (width 0.2))
+    (fp_line (start 3.44 1.85) (end 3.44 -1.85) (layer F.SilkS) (width 0.2))
+    (fp_line (start -3.44 1.85) (end 3.44 1.85) (layer F.SilkS) (width 0.2))
+    (fp_line (start -3.44 0.635) (end -3.44 1.85) (layer F.SilkS) (width 0.2))
+    (fp_line (start 3.325 1.85) (end -3.325 1.85) (layer Dwgs.User) (width 0.1))
+    (fp_line (start 3.325 -1.85) (end 3.325 1.85) (layer Dwgs.User) (width 0.1))
+    (fp_line (start -3.325 -1.85) (end 3.325 -1.85) (layer Dwgs.User) (width 0.1))
+    (fp_line (start -3.325 1.85) (end -3.325 -1.85) (layer Dwgs.User) (width 0.1))
+    (fp_line (start 3.575 2.1) (end -3.575 2.1) (layer Dwgs.User) (width 0.05))
+    (fp_line (start 3.575 -2.1) (end 3.575 2.1) (layer Dwgs.User) (width 0.05))
+    (fp_line (start -3.575 -2.1) (end 3.575 -2.1) (layer Dwgs.User) (width 0.05))
     (fp_line (start -3.575 2.1) (end -3.575 -2.1) (layer Dwgs.User) (width 0.05))
-    (fp_line (start -3.575 -2.1) (end 3.575 -2.1) (layer Dwgs.User) (width 0.05))
-    (fp_line (start 3.575 -2.1) (end 3.575 2.1) (layer Dwgs.User) (width 0.05))
-    (fp_line (start 3.575 2.1) (end -3.575 2.1) (layer Dwgs.User) (width 0.05))
-    (fp_line (start -3.325 1.85) (end -3.325 -1.85) (layer Dwgs.User) (width 0.1))
-    (fp_line (start -3.325 -1.85) (end 3.325 -1.85) (layer Dwgs.User) (width 0.1))
-    (fp_line (start 3.325 -1.85) (end 3.325 1.85) (layer Dwgs.User) (width 0.1))
-    (fp_line (start 3.325 1.85) (end -3.325 1.85) (layer Dwgs.User) (width 0.1))
-    (fp_line (start -3.44 0.635) (end -3.44 1.85) (layer F.SilkS) (width 0.2))
-    (fp_line (start -3.44 1.85) (end 3.44 1.85) (layer F.SilkS) (width 0.2))
-    (fp_line (start 3.44 1.85) (end 3.44 -1.85) (layer F.SilkS) (width 0.2))
-    (fp_line (start 3.44 -1.85) (end -2.54 -1.85) (layer F.SilkS) (width 0.2))
     (pad 10 thru_hole circle (at 2.54 -0.635 90) (size 1.1 1.1) (drill 0.7) (layers *.Cu *.Mask F.SilkS))
     (pad 9 thru_hole circle (at 2.54 0.635 90) (size 1.1 1.1) (drill 0.7) (layers *.Cu *.Mask F.SilkS))
@@
       (effects (font (size 1.27 1.27) (thickness 0.254)))
     )
+    (fp_line (start 3.44 -1.85008) (end -2.54 -1.85008) (layer F.SilkS) (width 0.2))
+    (fp_line (start 3.44 1.84992) (end 3.44 -1.85008) (layer F.SilkS) (width 0.2))
+    (fp_line (start -3.44 1.84992) (end 3.44 1.84992) (layer F.SilkS) (width 0.2))
+    (fp_line (start -3.44 0.63492) (end -3.44 1.84992) (layer F.SilkS) (width 0.2))
+    (fp_line (start 3.325 1.84992) (end -3.325 1.84992) (layer Dwgs.User) (width 0.1))
+    (fp_line (start 3.325 -1.85008) (end 3.325 1.84992) (layer Dwgs.User) (width 0.1))
+    (fp_line (start -3.325 -1.85008) (end 3.325 -1.85008) (layer Dwgs.User) (width 0.1))
+    (fp_line (start -3.325 1.84992) (end -3.325 -1.85008) (layer Dwgs.User) (width 0.1))
+    (fp_line (start 3.575 2.09992) (end -3.575 2.09992) (layer Dwgs.User) (width 0.05))
+    (fp_line (start 3.575 -2.095) (end 3.575 2.105) (layer Dwgs.User) (width 0.05))
+    (fp_line (start -3.575 -2.095) (end 3.575 -2.095) (layer Dwgs.User) (width 0.05))
     (fp_line (start -3.575 2.105) (end -3.575 -2.095) (layer Dwgs.User) (width 0.05))
-    (fp_line (start -3.575 -2.095) (end 3.575 -2.095) (layer Dwgs.User) (width 0.05))
-    (fp_line (start 3.575 -2.095) (end 3.575 2.105) (layer Dwgs.User) (width 0.05))
-    (fp_line (start 3.575 2.09992) (end -3.575 2.09992) (layer Dwgs.User) (width 0.05))
-    (fp_line (start -3.325 1.84992) (end -3.325 -1.85008) (layer Dwgs.User) (width 0.1))
-    (fp_line (start -3.325 -1.85008) (end 3.325 -1.85008) (layer Dwgs.User) (width 0.1))
-    (fp_line (start 3.325 -1.85008) (end 3.325 1.84992) (layer Dwgs.User) (width 0.1))
-    (fp_line (start 3.325 1.84992) (end -3.325 1.84992) (layer Dwgs.User) (width 0.1))
-    (fp_line (start -3.44 0.63492) (end -3.44 1.84992) (layer F.SilkS) (width 0.2))
-    (fp_line (start -3.44 1.84992) (end 3.44 1.84992) (layer F.SilkS) (width 0.2))
-    (fp_line (start 3.44 1.84992) (end 3.44 -1.85008) (layer F.SilkS) (width 0.2))
-    (fp_line (start 3.44 -1.85008) (end -2.54 -1.85008) (layer F.SilkS) (width 0.2))
     (pad 10 thru_hole circle (at 2.54 -0.63508 90) (size 1.1 1.1) (drill 0.7) (layers *.Cu *.Mask F.SilkS)
       (net 1 GND))
@@
       (effects (font (size 1 1) (thickness 0.15)))
     )
+    (fp_line (start -0.635 -1.27) (end 1.27 -1.27) (layer F.Fab) (width 0.1))
+    (fp_line (start 1.27 -1.27) (end 1.27 19.05) (layer F.Fab) (width 0.1))
+    (fp_line (start 1.27 19.05) (end -1.27 19.05) (layer F.Fab) (width 0.1))
+    (fp_line (start -1.27 19.05) (end -1.27 -0.635) (layer F.Fab) (width 0.1))
+    (fp_line (start -1.27 -0.635) (end -0.635 -1.27) (layer F.Fab) (width 0.1))
+    (fp_line (start -1.33 19.11) (end 1.33 19.11) (layer F.SilkS) (width 0.12))
+    (fp_line (start -1.33 1.27) (end -1.33 19.11) (layer F.SilkS) (width 0.12))
+    (fp_line (start 1.33 1.27) (end 1.33 19.11) (layer F.SilkS) (width 0.12))
+    (fp_line (start -1.33 1.27) (end 1.33 1.27) (layer F.SilkS) (width 0.12))
+    (fp_line (start -1.33 0) (end -1.33 -1.33) (layer F.SilkS) (width 0.12))
+    (fp_line (start -1.33 -1.33) (end 0 -1.33) (layer F.SilkS) (width 0.12))
+    (fp_line (start -1.8 -1.8) (end -1.8 19.55) (layer F.CrtYd) (width 0.05))
+    (fp_line (start -1.8 19.55) (end 1.8 19.55) (layer F.CrtYd) (width 0.05))
+    (fp_line (start 1.8 19.55) (end 1.8 -1.8) (layer F.CrtYd) (width 0.05))
     (fp_line (start 1.8 -1.8) (end -1.8 -1.8) (layer F.CrtYd) (width 0.05))
-    (fp_line (start 1.8 19.55) (end 1.8 -1.8) (layer F.CrtYd) (width 0.05))
-    (fp_line (start -1.8 19.55) (end 1.8 19.55) (layer F.CrtYd) (width 0.05))
-    (fp_line (start -1.8 -1.8) (end -1.8 19.55) (layer F.CrtYd) (width 0.05))
-    (fp_line (start -1.33 -1.33) (end 0 -1.33) (layer F.SilkS) (width 0.12))
-    (fp_line (start -1.33 0) (end -1.33 -1.33) (layer F.SilkS) (width 0.12))
-    (fp_line (start -1.33 1.27) (end 1.33 1.27) (layer F.SilkS) (width 0.12))
-    (fp_line (start 1.33 1.27) (end 1.33 19.11) (layer F.SilkS) (width 0.12))
-    (fp_line (start -1.33 1.27) (end -1.33 19.11) (layer F.SilkS) (width 0.12))
-    (fp_line (start -1.33 19.11) (end 1.33 19.11) (layer F.SilkS) (width 0.12))
-    (fp_line (start -1.27 -0.635) (end -0.635 -1.27) (layer F.Fab) (width 0.1))
-    (fp_line (start -1.27 19.05) (end -1.27 -0.635) (layer F.Fab) (width 0.1))
-    (fp_line (start 1.27 19.05) (end -1.27 19.05) (layer F.Fab) (width 0.1))
-    (fp_line (start 1.27 -1.27) (end 1.27 19.05) (layer F.Fab) (width 0.1))
-    (fp_line (start -0.635 -1.27) (end 1.27 -1.27) (layer F.Fab) (width 0.1))
     (fp_text user %R (at 0 8.89) (layer F.Fab) hide
       (effects (font (size 1 1) (thickness 0.15)))
@@
       (effects (font (size 1 1) (thickness 0.15)))
     )
+    (fp_line (start -0.8 0.4) (end -0.8 -0.4) (layer F.Fab) (width 0.1))
+    (fp_line (start -0.8 -0.4) (end 0.8 -0.4) (layer F.Fab) (width 0.1))
+    (fp_line (start 0.8 -0.4) (end 0.8 0.4) (layer F.Fab) (width 0.1))
+    (fp_line (start 0.8 0.4) (end -0.8 0.4) (layer F.Fab) (width 0.1))
+    (fp_line (start -0.146267 -0.51) (end 0.146267 -0.51) (layer F.SilkS) (width 0.12))
+    (fp_line (start -0.146267 0.51) (end 0.146267 0.51) (layer F.SilkS) (width 0.12))
+    (fp_line (start -1.65 0.73) (end -1.65 -0.73) (layer F.CrtYd) (width 0.05))
+    (fp_line (start -1.65 -0.73) (end 1.65 -0.73) (layer F.CrtYd) (width 0.05))
+    (fp_line (start 1.65 -0.73) (end 1.65 0.73) (layer F.CrtYd) (width 0.05))
     (fp_line (start 1.65 0.73) (end -1.65 0.73) (layer F.CrtYd) (width 0.05))
-    (fp_line (start 1.65 -0.73) (end 1.65 0.73) (layer F.CrtYd) (width 0.05))
-    (fp_line (start -1.65 -0.73) (end 1.65 -0.73) (layer F.CrtYd) (width 0.05))
-    (fp_line (start -1.65 0.73) (end -1.65 -0.73) (layer F.CrtYd) (width 0.05))
-    (fp_line (start -0.146267 0.51) (end 0.146267 0.51) (layer F.SilkS) (width 0.12))
-    (fp_line (start -0.146267 -0.51) (end 0.146267 -0.51) (layer F.SilkS) (width 0.12))
-    (fp_line (start 0.8 0.4) (end -0.8 0.4) (layer F.Fab) (width 0.1))
-    (fp_line (start 0.8 -0.4) (end 0.8 0.4) (layer F.Fab) (width 0.1))
-    (fp_line (start -0.8 -0.4) (end 0.8 -0.4) (layer F.Fab) (width 0.1))
-    (fp_line (start -0.8 0.4) (end -0.8 -0.4) (layer F.Fab) (width 0.1))
     (fp_text user %R (at 0.02 -1.22) (layer F.Fab) hide
       (effects (font (size 0.4 0.4) (thickness 0.06)))
