File: PCB/controller/controller.kicad_pcb (KiCad board)
At the start: 2 copper layers, 54 x 71 mm, 8 parts, among them J1 Conn_01x12_Female, J2 Conn_01x16_Female, J3 Conn_01x16_Female, U1 Adafruit_Feather_nRF52840

Commit message: udated by FZ
Parts:
- moved H1 0.50 mm to (122.5, 58.0)
- moved H2 0.50 mm to (122.5, 123.0)
Other:
- board size 54 x 71 mm -> 54.5 x 71 mm
- board text added: "10"
- board text added: "11"
- board text added: "12"
- board text added: "13"
- board text added: "2"
- board text added: "3.3V"
- board text added: "5"
- board text added: "6"
- board text added: "9"
- board text added: "A0"
- board text added: "A1"
- board text added: "A2"
- board text added: "A3"
- board text added: "A4"
- board text added: "A5"
- board text added: "AstroAnt Central station"
- board text added: "GND"
