File: PCB/impedance_measurement/impedance_measurement.sch (KiCad schematic (older format))
At the start: 26 parts, among them J1 RF_SMD, J2 RF_SMD, J3 20021321-00014C1LF, J4 20021321-00010C4LF, U1 AD8606ARZ, U2 AD5933YRSZ-REEL7, U3 ADP150AUJZ-3.0-R7

Commit message: udated by FZ
Parts:
- added C9: 0.1uF, Capacitor_SMD:C_0603_1608Metric_Pad1.08x0.95mm_HandSolder, symbol Device:C_Small
- added R11: 100, Resistor_SMD:R_0805_2012Metric_Pad1.20x1.40mm_HandSolder, symbol Device:R_Small
- added S1: ADG849YKSZ-REEL7, SamacSys_Parts:SOT65P210X110-6N, symbol SamacSys_Parts:ADG849YKSZ-REEL7
Connections:
- net GND: now also J3.1, C9.1, S1.3 (GND)
- net GNDREF: no longer J3.1
- net SIG_IN: now also R11.2
- net SIG_OUT: now also S1.5 (D); no longer J1.1
- net VDD: now also C9.2, S1.2 (VDD)
- net Cali_switch: now reaches J3.10
- net Cali_switch: now also S1.1 (IN)
- new net: R11.1, S1.4 (S1)
- new net SIG_OUT_probe: J1.1, S1.6 (S2)
- no-connect marks 21 -> 20
Other:
- moved on the sheet: C1, C2, C3, C4, C5, C6, C7, C8, FB1, J1, J2, J3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

Commit message: udated by FZ
Parts:
- C1: value 10uF -> 0.1uF
- C2: value 0.1uF -> 10uF
Changed lines of the file:
@@
 P 3400 1900
 F 0 "C2" H 3510 1830 50  0000 C CNN
-F 1 "0.1uF" H 3530 1990 50  0000 C CNN
+F 1 "10uF" H 3530 1990 50  0000 C CNN
 F 2 "Capacitor_SMD:C_0603_1608Metric_Pad1.08x0.95mm_HandSolder" H 3400 1900 50  0001 C CNN
 F 3 "~" H 3400 1900 50  0001 C CNN
@@
 P 3100 1900
 F 0 "C1" H 3210 1830 50  0000 C CNN
-F 1 "10uF" H 3230 1990 50  0000 C CNN
+F 1 "0.1uF" H 3230 1990 50  0000 C CNN
 F 2 "Capacitor_SMD:C_0603_1608Metric_Pad1.08x0.95mm_HandSolder" H 3100 1900 50  0001 C CNN
 F 3 "~" H 3100 1900 50  0001 C CNN
